Commit message: Updated HyQ model

File: hyq.urdf (robot description, URDF)
Before this commit: robot hyq, 17 links, 16 joints
Links:
- link LF_HIP_FE: geometry collision mesh filename=ycyl-r0.01-l0.35.obj; visual mesh filename=ycyl-r0.01-l0.35.obj
- link LF_KNEE: geometry collision mesh filename=ycyl-r0.01-l0.33.obj; visual mesh filename=ycyl-r0.01-l0.33.obj
- link LH_HIP_FE: geometry collision mesh filename=ycyl-r0.01-l0.35.obj; visual mesh filename=ycyl-r0.01-l0.35.obj
- link LH_KNEE: geometry collision mesh filename=ycyl-r0.01-l0.33.obj; visual mesh filename=ycyl-r0.01-l0.33.obj
- link RF_HIP_FE: geometry collision mesh filename=ycyl-r0.01-l0.35.obj; visual mesh filename=ycyl-r0.01-l0.35.obj
- link RF_KNEE: geometry collision mesh filename=ycyl-r0.01-l0.33.obj; visual mesh filename=ycyl-r0.01-l0.33.obj
- link RH_HIP_FE: geometry collision mesh filename=ycyl-r0.01-l0.35.obj; visual mesh filename=ycyl-r0.01-l0.35.obj
- link RH_KNEE: geometry collision mesh filename=ycyl-r0.01-l0.33.obj; visual mesh filename=ycyl-r0.01-l0.33.obj

Commit message: Updated HyQ model and added simple PD controller

File: hyq.urdf (robot description, URDF)
Before this commit: robot hyq, 17 links, 16 joints
Links:
- link LF_HIP_FE: geometry collision cylinder length=0.35 radius=0.01; visual cylinder length=0.35 radius=0.01
- link LF_KNEE: geometry collision cylinder length=0.33 radius=0.01; visual cylinder length=0.33 radius=0.01
- link LH_HIP_FE: geometry collision cylinder length=0.35 radius=0.01; visual cylinder length=0.35 radius=0.01
- link LH_KNEE: geometry collision cylinder length=0.33 radius=0.01; visual cylinder length=0.33 radius=0.01
- link RF_HIP_FE: geometry collision cylinder length=0.35 radius=0.01; visual cylinder length=0.35 radius=0.01
- link RF_KNEE: geometry collision cylinder length=0.33 radius=0.01; visual cylinder length=0.33 radius=0.01
- link RH_HIP_FE: geometry collision cylinder length=0.35 radius=0.01; visual cylinder length=0.35 radius=0.01
- link RH_KNEE: geometry collision cylinder length=0.33 radius=0.01; visual mesh filename=ycyl-r0.01-l0.33.obj

Commit message: modifying htq controllers

File: hyq.urdf (robot description, URDF)
Before this commit: robot hyq, 17 links, 16 joints
Links:
- link LF_FOOT: geometry collision box size=0.02 0.02 0.02; visual box size=0.02 0.02 0.02
- link LH_FOOT: geometry collision box size=0.02 0.02 0.02; visual box size=0.02 0.02 0.02
- link RF_FOOT: geometry collision box size=0.02 0.02 0.02; visual box size=0.02 0.02 0.02
- link RH_FOOT: geometry collision box size=0.02 0.02 0.02; visual box size=0.02 0.02 0.02
- link RH_KNEE: geometry collision box size=0.02 0.02 0.02; visual mesh filename=ycyl-r0.01-l0.33.obj
Joints:
- joint LF_HAA: limit lower=-1.571 upper=0.524 effort=100.000000 velocity=10.0 -> (none); type revolute -> continuous
- joint LF_HFE: limit lower=-0.873 upper=1.222 effort=100.000000 velocity=10.0 -> (none); type revolute -> continuous
- joint LF_KFE: limit lower=-2.443 upper=-0.349 effort=100.000000 velocity=10.0 -> (none); type revolute -> continuous
- joint LH_HAA: limit lower=-1.571 upper=0.524 effort=100.000000 velocity=10.0 -> (none); type revolute -> continuous
- joint LH_HFE: limit lower=-1.222 upper=0.873 effort=100.000000 velocity=10.0 -> (none); type revolute -> continuous
- joint LH_KFE: limit lower=0.349 upper=2.443 effort=100.000000 velocity=10.0 -> (none); type revolute -> continuous
- joint RF_HAA: limit lower=-1.571 upper=0.524 effort=100.000000 velocity=10.0 -> (none); type revolute -> continuous
- joint RF_HFE: limit lower=-0.873 upper=1.222 effort=100.000000 velocity=10.0 -> (none); type revolute -> continuous
- joint RF_KFE: limit lower=-2.443 upper=-0.349 effort=100.000000 velocity=10.0 -> (none); type revolute -> continuous
- joint RH_HAA: limit lower=-1.571 upper=0.524 effort=100.000000 velocity=10.0 -> (none); type revolute -> continuous
- joint RH_HFE: limit lower=-1.222 upper=0.873 effort=100.000000 velocity=10.0 -> (none); type revolute -> continuous
- joint RH_KFE: limit lower=0.349 upper=2.443 effort=100.000000 velocity=10.0 -> (none); type revolute -> continuous

Commit message: Updated hyq model and controller

File: hyq.urdf (robot description, URDF)
Before this commit: robot hyq, 17 links, 16 joints
Joints:
- joint LF_HAA: axis 0 0 1 -> 0 0 -1; origin xyz=0.3735 0.207 0.0 rpy=0 1.570796 3.141593 -> xyz=0.3735 0.207 0.0 rpy=0 1.5708 0
- joint LF_HFE: axis 0 0 1 -> 0 1 0; origin xyz=0.08 0.0 0.0 rpy=1.570796 0.0 0.0 -> xyz=0.08 0.0 0.0 rpy=0.0 -1.5708 0.0
- joint LF_KFE: axis 0 0 1 -> 0 1 0; origin xyz=0.35 0.0 0.0 rpy=0.0 0.0 0.0 -> xyz=0.0 0.0 -0.35 rpy=0.0 0.0 0.0
- joint LF_LLF: origin xyz=0.33 0.0 0.0 rpy=0.0 0.0 0.0 -> xyz=0 0 -0.33 rpy=0.0 0.0 0.0
- joint LH_HAA: axis 0 0 1 -> 0 0 -1; origin xyz=-0.3735 0.207 0.0 rpy=3.141593 1.570796 0.0 -> xyz=-0.3735 0.207 0.0 rpy=0 1.5708 0.0
- joint LH_HFE: axis 0 0 1 -> 0 1 0; origin xyz=0.08 0.0 0.0 rpy=1.570796 0.0 0.0 -> xyz=0.08 0.0 0.0 rpy=0 -1.570796 0.0
- joint LH_KFE: axis 0 0 1 -> 0 1 0; origin xyz=0.35 0.0 0.0 rpy=0.0 0.0 0.0 -> xyz=0 0 -0.35 rpy=0.0 0.0 0.0
- joint LH_LLF: origin xyz=0.33 0.0 0.0 rpy=0.0 -1.570796 -1.570796 -> xyz=0 0 -0.33 rpy=0.0 0 0
- joint RF_HAA: axis 0 0 1 -> 0 0 -1; origin xyz=0.3735 -0.207 0.0 rpy=0 1.570796 0 -> xyz=0.3735 -0.207 0.0 rpy=0 1.5708 0
- joint RF_HFE: axis 0 0 1 -> 0 1 0; origin xyz=0.08 0.0 0.0 rpy=-1.570796 0.0 0.0 -> xyz=0.08 0.0 0.0 rpy=0 -1.570796 0.0
- joint RF_KFE: axis 0 0 1 -> 0 1 0; origin xyz=0.35 0.0 0.0 rpy=0.0 0.0 0.0 -> xyz=0.0 0.0 -0.35 rpy=0.0 0.0 0.0
- joint RF_LLF: origin xyz=0.33 0.0 0.0 rpy=0.0 -1.570796 -1.570796 -> xyz=0 0 -0.33 rpy=0.0 0 0
- joint RH_HAA: axis 0 0 1 -> 0 0 -1; origin xyz=-0.3735 -0.207 0.0 rpy=0.0 1.570796 0.0 -> xyz=-0.3735 -0.207 0.0 rpy=0.0 1.5708 0.0
- joint RH_HFE: axis 0 0 1 -> 0 1 0; origin xyz=0.08 0.0 0.0 rpy=-1.570796 0.0 0.0 -> xyz=0.08 0.0 0.0 rpy=0 -1.570796 0.0
- joint RH_KFE: axis 0 0 1 -> 0 1 0; origin xyz=0.35 0.0 0.0 rpy=0.0 0.0 0.0 -> xyz=0 0 -0.35 rpy=0.0 0.0 0.0
- joint RH_LLF: origin xyz=0.33 0.0 0.0 rpy=0.0 -1.570796 -1.570796 -> xyz=0 0 -0.33 rpy=0.0 0 0
