Commit message: fixed lynx

File: links.urdf (robot description, URDF)
Before this commit: robot links, 14 links, 13 joints
Links:
- link ABDOMEN: mass 25.000000 -> 3.0; geometry collision box size=0.0355 0.101 0.0356; visual box size=0.0860 0.101 0.0356
- link LF_HIP: mass 1.772000 -> 1.0
- link LF_LLEG: mass 1.600000 -> 1.0
- link LF_ULEG: mass 1.772 -> 1.0
- link LH_HIP: mass 1.772000 -> 1.0; geometry collision box size=0.0611 0.0402 0.041; visual box size=0.0611 0.0402 0.041
- link LH_LLEG: mass 1.600000 -> 1.0
- link LH_ULEG: mass 2.482000 -> 1.0
- link RF_HIP: mass 1.772000 -> 1.0
- link RF_LLEG: mass 1.600000 -> 1.0
- link RF_ULEG: mass 2.482000 -> 1.0
- link RH_HIP: mass 1.772000 -> 1.0; geometry collision box size=0.0611 0.0402 0.041; visual box size=0.0611 0.0402 0.041
- link RH_LLEG: mass 1.600000 -> 1.0
- link RH_ULEG: mass 2.482000 -> 1.0
- link THORAX: mass 25.000000 -> 2.0
Joints:
- joint BODY_JOINT: origin xyz=-0.0505 0.0 0.0 rpy=0.0 0.0 3.1415 -> xyz=0.043 0.0 0.0 rpy=0.0 0.0 0.0
- joint LF_HIP_AA: origin xyz=0.0355 0.0505 0.0 rpy=0 0 0 -> xyz=0.043 0.0475 0.0 rpy=0 0 0
- joint LH_HIP_AA: origin xyz=0.0355 0.0505 0.0 rpy=0 0 0.0 -> xyz=-0.043 0.0475 0.0 rpy=0 0 3.1416
- joint LH_HIP_FE: origin xyz=0.0505 0.0 0.0 rpy=0 0 0.0 -> xyz=0.0611 0.0 0.0 rpy=0 0 0
- joint RF_HIP_AA: origin xyz=0.0355 -0.0505 0.0 rpy=0 0 0 -> xyz=0.043 -0.0475 0.0 rpy=0 0 0
- joint RH_HIP_AA: origin xyz=0.0355 -0.0505 0.0 rpy=0.0 0.0 0.0 -> xyz=-0.043 -0.0475 0.0 rpy=0 0 3.1416
- joint RH_HIP_FE: origin xyz=0.0505 0.0 0.0 rpy=0 0 0 -> xyz=0.0611 0.0 0.0 rpy=0 0 0

Commit message: updated LYNX

File: links.urdf (robot description, URDF)
Before this commit: robot links, 14 links, 13 joints
Joints:
- joint BODY_JOINT: type continuous -> revolute
- joint LF_HIP_AA: type continuous -> revolute
- joint LF_HIP_FE: type continuous -> revolute
- joint LF_LEG_FE: type continuous -> revolute
- joint LH_HIP_AA: type continuous -> revolute
- joint LH_HIP_FE: type continuous -> revolute
- joint LH_LEG_FE: type continuous -> revolute
- joint RF_HIP_AA: type continuous -> revolute
- joint RF_HIP_FE: type continuous -> revolute
- joint RF_LEG_FE: type continuous -> revolute
- joint RH_HIP_AA: type continuous -> revolute
- joint RH_HIP_FE: type continuous -> revolute
- joint RH_LEG_FE: type continuous -> revolute

Commit message: links foot rotation, contact poly and points added

File: links.urdf (robot description, URDF)
Before this commit: robot links, 14 links, 13 joints
Links:
- link ABDOMEN: geometry collision box size=0.0860 0.101 0.0356; visual box size=0.0860 0.101 0.0356

Commit message: lynx walking in sim (kinematic mode is enabled)

File: links.urdf (robot description, URDF)
Before this commit: robot links, 14 links, 13 joints
Links:
- link ABDOMEN: mass 3.0 -> 10.0
- link THORAX: mass 2.0 -> 10.0

Commit message: for now controller is commented out to demonstrate a bug

File: links.urdf (robot description, URDF)
Before this commit: robot links, 14 links, 13 joints
Links:
- link ABDOMEN: mass 10.0 -> 2.01; geometry collision box size=0.860 1.01 0.356; visual box size=0.860 1.01 0.356
- link LF_HIP: mass 1.0 -> 0.63; geometry collision box size=0.505 0.355 0.356; visual box size=0.505 0.355 0.356
- link LF_LLEG: mass 1.0 -> 0.63; geometry collision box size=0.8 0.1 0.1; visual box size=0.8 0.1 0.1
- link LF_ULEG: mass 1.0 -> 0.63; geometry collision box size=0.505 0.355 0.356; visual box size=0.505 0.355 0.356
- link LH_HIP: mass 1.0 -> 1.26; geometry collision box size=0.611 0.402 0.41; visual box size=0.611 0.402 0.41
- link LH_LLEG: mass 1.0 -> 0.63; geometry collision box size=0.8 0.1 0.1; visual box size=0.8 0.1 0.1
- link LH_ULEG: mass 1.0 -> 0.63; geometry collision box size=0.505 0.355 0.356; visual box size=0.505 0.355 0.356
- link RF_HIP: mass 1.0 -> 0.63; geometry collision box size=0.505 0.355 0.356; visual box size=0.505 0.355 0.356
- link RF_LLEG: mass 1.0 -> 0.63; geometry collision box size=0.8 0.1 0.1; visual box size=0.8 0.1 0.1
- link RF_ULEG: mass 1.0 -> 0.63; geometry collision box size=0.505 0.355 0.356; visual box size=0.505 0.355 0.356
- link RH_HIP: mass 1.0 -> 1.26; geometry collision box size=0.611 0.402 0.41; visual box size=0.611 0.402 0.41
- link RH_LLEG: mass 1.0 -> 0.63; geometry collision box size=0.8 0.1 0.1; visual box size=0.8 0.1 0.1
- link RH_ULEG: mass 1.0 -> 0.63; geometry collision box size=0.505 0.355 0.356; visual box size=0.505 0.355 0.356
- link THORAX: mass 10.0 -> 1.34; geometry collision box size=0.355 1.01 0.356; visual box size=0.355 1.01 0.356
Joints:
- joint BODY_JOINT: origin xyz=0.043 0.0 0.0 rpy=0.0 0.0 0.0 -> xyz=0.43 0.0 0.0 rpy=0.0 0.0 0.0; type revolute -> continuous
- joint LF_HIP_AA: origin xyz=0.043 0.0475 0.0 rpy=0 0 0 -> xyz=0.43 0.475 0.0 rpy=0 0 0; type revolute -> continuous
- joint LF_HIP_FE: origin xyz=0.0505 0.0 0.0 rpy=0 0 0.0 -> xyz=0.505 0.0 0.0 rpy=0 0.78539 0.0; type revolute -> continuous
- joint LF_LEG_FE: origin xyz=0.0505 0.0 0.0 rpy=0.0 0.0 0.0 -> xyz=0.505 0.0 0.0 rpy=0.0 0.0 0.0; type revolute -> continuous
- joint LH_HIP_AA: origin xyz=-0.043 0.0475 0.0 rpy=0 0 3.1416 -> xyz=-0.43 0.475 0.0 rpy=0 0 3.1416; type revolute -> continuous
- joint LH_HIP_FE: origin xyz=0.0611 0.0 0.0 rpy=0 0 0 -> xyz=0.611 0.0 0.0 rpy=0 0.78539 0; type revolute -> continuous
- joint LH_LEG_FE: origin xyz=0.0505 0.0 0.0 rpy=0.0 0.0 0.0 -> xyz=0.505 0.0 0.0 rpy=0.0 0.0 0.0; type revolute -> continuous
- joint RF_HIP_AA: origin xyz=0.043 -0.0475 0.0 rpy=0 0 0 -> xyz=0.43 -0.475 0.0 rpy=0 0 0; type revolute -> continuous
- joint RF_HIP_FE: origin xyz=0.0505 0.0 0.0 rpy=0 0 0.0 -> xyz=0.505 0.0 0.0 rpy=0 0.78539 0.0; type revolute -> continuous
- joint RF_LEG_FE: origin xyz=0.0505 0.0 0.0 rpy=0.0 0.0 0.0 -> xyz=0.505 0.0 0.0 rpy=0.0 0.0 0.0; type revolute -> continuous
- joint RH_HIP_AA: origin xyz=-0.043 -0.0475 0.0 rpy=0 0 3.1416 -> xyz=-0.43 -0.475 0.0 rpy=0 0 3.1416; type revolute -> continuous
- joint RH_HIP_FE: origin xyz=0.0611 0.0 0.0 rpy=0 0 0 -> xyz=0.611 0.0 0.0 rpy=0 0.78539 0; type revolute -> continuous
- joint RH_LEG_FE: origin xyz=0.0505 0.0 0.0 rpy=0 0.0 0.0 -> xyz=0.505 0.0 0.0 rpy=0 0.0 0.0; type revolute -> continuous

Commit message: robot 0 state is in standing postition

File: links.urdf (robot description, URDF)
Before this commit: robot links, 14 links, 13 joints
Joints:
- joint LF_LEG_FE: origin xyz=0.0505 0.0 0.0 rpy=0.0 0.0 0.0 -> xyz=0.0505 0.0 0.0 rpy=0.0 1.5708 0.0
- joint LH_LEG_FE: origin xyz=0.0505 0.0 0.0 rpy=0.0 0.0 0.0 -> xyz=0.0505 0.0 0.0 rpy=0.0 1.5708 0.0
- joint RF_LEG_FE: origin xyz=0.0505 0.0 0.0 rpy=0.0 0.0 0.0 -> xyz=0.0505 0.0 0.0 rpy=0.0 1.5708 0.0
- joint RH_LEG_FE: origin xyz=0.0505 0.0 0.0 rpy=0 0.0 0.0 -> xyz=0.0505 0.0 0.0 rpy=0 1.5708 0.0

Commit message: energy calculation code added

File: links.urdf (robot description, URDF)
Before this commit: robot links, 14 links, 13 joints
Joints:
- joint BODY_JOINT: origin xyz=0.043 0.0 0.0 rpy=0.0 0.0 0.0 -> xyz=0.043 0.0 0.0 rpy=0 0 0
- joint LF_HIP_FE: origin xyz=0.0505 0.0 0.0 rpy=0 0.78539 0.0 -> xyz=0.0505 0.0 0.0 rpy=0 0.78539 0
- joint LF_LEG_FE: origin xyz=0.0505 0.0 0.0 rpy=0.0 1.5708 0.0 -> xyz=0.0505 0.0 0.0 rpy=0 1.5708 0
- joint LH_LEG_FE: origin xyz=0.0505 0.0 0.0 rpy=0.0 1.5708 0.0 -> xyz=0.0505 0.0 0.0 rpy=0 1.5708 0
- joint RF_HIP_FE: origin xyz=0.0505 0.0 0.0 rpy=0 0.78539 0.0 -> xyz=0.0505 0.0 0.0 rpy=0 0.78539 0
- joint RF_LEG_FE: origin xyz=0.0505 0.0 0.0 rpy=0.0 1.5708 0.0 -> xyz=0.0505 0.0 0.0 rpy=0 1.5708 0

Commit message: added analytical IK code

File: links.urdf (robot description, URDF)
Before this commit: robot links, 14 links, 13 joints
Joints:
- joint LF_HIP_FE: origin xyz=0.0505 0.0 0.0 rpy=0 0.78539 0 -> xyz=0.0505 0.0 0.0 rpy=0 0 0
- joint LH_HIP_FE: origin xyz=0.0611 0.0 0.0 rpy=0 0.78539 0 -> xyz=0.0611 0.0 0.0 rpy=0 0 0
- joint RF_HIP_FE: origin xyz=0.0505 0.0 0.0 rpy=0 0.78539 0 -> xyz=0.0505 0.0 0.0 rpy=0 0 0
- joint RH_HIP_FE: origin xyz=0.0611 0.0 0.0 rpy=0 0.78539 0 -> xyz=0.0611 0.0 0.0 rpy=0 0 0
- joint RH_LEG_FE: origin xyz=0.0505 0.0 0.0 rpy=0 1.5708 0.0 -> xyz=0.0505 0.0 0.0 rpy=0 0 0.0

Commit message: IK working (must select a 'best' solution somehow)

File: links.urdf (robot description, URDF)
Before this commit: robot links, 14 links, 13 joints
Joints:
- joint LF_LEG_FE: origin xyz=0.0505 0.0 0.0 rpy=0 1.5708 0 -> xyz=0.0505 0.0 0.0 rpy=0 0 0
- joint LH_LEG_FE: origin xyz=0.0505 0.0 0.0 rpy=0 1.5708 0 -> xyz=0.0505 0.0 0.0 rpy=0 0 0
- joint RF_LEG_FE: origin xyz=0.0505 0.0 0.0 rpy=0 1.5708 0 -> xyz=0.0505 0.0 0.0 rpy=0 0 0

Commit message: added links feet

File: links.urdf (robot description, URDF)
Before this commit: robot links, 14 links, 13 joints
Links:
- added link LF_FOOT, mass 0.001; collision sphere radius=0.005; visual sphere radius=0.005
- added link LH_FOOT, mass 0.001; collision sphere radius=0.005; visual sphere radius=0.005
- added link RF_FOOT, mass 0.001; collision sphere radius=0.005; visual sphere radius=0.005
- added link RH_FOOT, mass 0.001; collision sphere radius=0.005; visual sphere radius=0.005
Joints:
- added joint LF_ANKLE: type fixed, parent LF_LLEG, child LF_FOOT, origin xyz=0.04 0.0 0.0 rpy=0 0 0.0
- added joint LH_ANKLE: type fixed, parent LH_LLEG, child LH_FOOT, origin xyz=0.04 0.0 0.0 rpy=0 0 0.0
- added joint RF_ANKLE: type fixed, parent RF_LLEG, child RF_FOOT, origin xyz=0.04 0.0 0.0 rpy=0 0 0.0
- added joint RH_ANKLE: type fixed, parent RH_LLEG, child RH_FOOT, origin xyz=0.04 0.0 0.0 rpy=0 0 0.0

Commit message: 4-leg IK functioning

File: links.urdf (robot description, URDF)
Before this commit: robot links, 18 links, 17 joints
Links:
- link RH_LLEG: mass 0.063 -> 0.05

Commit message: now using moby format for lynx (see lynx-model.xml)

File: links.urdf (robot description, URDF)
Before this commit: robot links, 18 links, 17 joints
Joints:
- joint LF_ANKLE: origin xyz=0.04 0.0 0.0 rpy=0 0 0.0 -> xyz=0.08 0.0 0.0 rpy=0 0 0.0
- joint LH_ANKLE: origin xyz=0.04 0.0 0.0 rpy=0 0 0.0 -> xyz=0.08 0.0 0.0 rpy=0 0 0.0
- joint RF_ANKLE: origin xyz=0.04 0.0 0.0 rpy=0 0 0.0 -> xyz=0.08 0.0 0.0 rpy=0 0 0.0
- joint RH_ANKLE: origin xyz=0.04 0.0 0.0 rpy=0 0 0.0 -> xyz=0.08 0.0 0.0 rpy=0 0 0.0
