Commit message: atlas sdf

File: Examples/Quadruped/MODELS/atlas_simple_shapes.urdf (robot description, URDF)
Before this commit: robot drc_skeleton, 13 links, 12 joints
Joints:
- joint l_leg_kny4: limit lower=0 upper=2.45 effort=400 velocity=12 -> (none); type revolute -> continuous
- joint l_leg_lax6: limit lower=-0.436 upper=0.436 effort=90 velocity=12 -> (none); type revolute -> continuous
- joint l_leg_lhy3: limit lower=-1.75 upper=0.524 effort=260 velocity=12 -> (none); type revolute -> continuous
- joint l_leg_mhx2: limit lower=-0.47 upper=0.495 effort=180 velocity=12 -> (none); type revolute -> continuous
- joint l_leg_uay5: limit lower=-0.9 upper=0.698 effort=220 velocity=12 -> (none); type revolute -> continuous
- joint l_leg_uhz1: limit lower=-0.32 upper=1.14 effort=110 velocity=12 -> (none); type revolute -> continuous
- joint r_leg_kny4: limit lower=0 upper=2.45 effort=400 velocity=12 -> (none); type revolute -> continuous
- joint r_leg_lax6: limit lower=-0.436 upper=0.436 effort=90 velocity=12 -> (none); type revolute -> continuous
- joint r_leg_lhy3: limit lower=-1.745 upper=0.524 effort=260 velocity=12 -> (none); type revolute -> continuous
- joint r_leg_mhx2: limit lower=-0.495 upper=0.47 effort=180 velocity=12 -> (none); type revolute -> continuous
- joint r_leg_uay5: limit lower=-0.9 upper=0.698 effort=220 velocity=12 -> (none); type revolute -> continuous
- joint r_leg_uhz1: limit lower=-1.14 upper=0.32 effort=110 velocity=12 -> (none); type revolute -> continuous
